File: ptSolarHF/ptSolarHF.kicad_pcb (KiCad board)
At the start: 4 copper layers, 38.5 x 73.5 mm, 55 parts, among them J1 6 Pin Male Header, J2 Programming, Q5 DMP2004K-7, U1 LP3985IM5-3.3/NOPB, U2 ATMega 328p-AU, U3 Si5351A-B-GT, U4 ATGM336H-5N31, U5 APX803S (SOT23SA), Y1 8MHz, Y2 Crystal_GND24

Commit message: Tweaks to proof of concept. Updates to Schematics.
Parts:
- added C15: 100nF, Capacitor_SMD:C_0805_2012Metric, F.Cu at (124.1, 93.0)
- added R10: 150k, Resistor_SMD:R_0805_2012Metric, F.Cu at (124.0, 99.2)
- C16, C19: value 54pF -> 150pF
- L1: value 381nH -> 270nF
- L2: value 612nH -> 270nH
- L3: value 381nH -> 270nH
- Y2: value Crystal_GND24 -> 27MHz Xtal - 7M-27.000MEEQ-T
- renumbered C14 to C13, C13 to C14, R23 to R11
Connections:
- C16 pad 2: Net-(U3-CLK0) -> Net-(C15-Pad2)
- L1 pad 1: Net-(U3-CLK0) -> Net-(C15-Pad2)

Commit message: Finalizing PCB v1.0.1
Parts:
- removed ANT2a1, ANT2b1: VHF Test Point, Custom DS:Small Test Point Pin
- moved R10 31.7 mm to (143.2, 74.0)
- moved C15 21.3 mm to (144.1, 85.6)
- moved C4 7.86 mm to (156.2, 82.8), turned to -90 degrees
- moved C13 2.83 mm to (147.6, 85.6), turned to 0 degrees
- moved C18 1.46 mm to (148.4, 76.6)
- moved L1 1.40 mm to (144.8, 82.6)
- moved L3 1.32 mm to (144.8, 76.8)
- moved C16 1.21 mm to (148.6, 83.2)
- moved C19 0.90 mm to (147.0, 74.0)
- moved C17 0.82 mm to (147.0, 80.6)
- moved L2 0.40 mm to (143.6, 79.8)
Routing:
- net +3.3V: track 60.7 -> 55.3 mm
- net Net-(C15-Pad2): track 0.00 -> 4.64 mm
- net Net-(U3-CLK0): track 5.25 -> 2.81 mm
- net +BATT: track 144.7 -> 142.8 mm
- net Net-(C17-Pad2): track 6.11 -> 4.31 mm
- net GND: track 34.6 -> 33.2 mm, vias 50 -> 146
Other:
- board text added: "PV1"
- board text added: "PV2"
- board text added: "ptSolarHF Tracker v1.0.1 Custom Digital Services, LLC www.custom-ds.com"
- board text removed: "ptSolarHF Tracker v1.0.0 Custom Digital Services, LLC www.custom-ds.com"
