File: ptSolarHF/ptSolarHF.kicad_pcb (KiCad board)
At the start: 4 copper layers, 38.5 x 73.5 mm, 55 parts, among them J1 6 Pin Male Header, J2 Programming, Q5 DMP2004K-7, U1 LP3985IM5-3.3/NOPB, U2 ATMega 328p-AU, U3 Si5351A-B-GT, U4 ATGM336H-5N31, U5 APX803S (SOT23SA), Y1 8MHz, Y2 27MHz Xtal - 7M-27.000MEEQ-T

Commit message: 26MHz TCXO and version 2.0.0 of PCB
Parts:
- added C22: 10nF, Capacitor_SMD:C_0805_2012Metric, F.Cu at (142.4, 91.2)
- added C23: 10nF, Capacitor_SMD:C_0805_2012Metric, F.Cu at (145.6, 94.2)
- C1: value 6V 1F -> 6V 0.5F
- C16, C19: value 150pF -> 180pF
- C17, C18: value 220pF -> 270pF
- L1: value 270nF -> 330nH
- L2: value 270nH -> 390nH
- L3: value 270nH -> 330nH
- R10: value 150k -> 10k
- Y2: value 27MHz Xtal - 7M-27.000MEEQ-T -> 26.000MHz TCXO; footprint Crystal:Crystal_SMD_3225-4Pin_3.2x2.5mm -> Oscillator:Oscillator_SMD_SeikoEpson_TG2520SMN-xxx-xxxxxx-4Pin_2.5x2.0mm
- moved Y2 1.57 mm to (145.6, 96.8), turned to 90 degrees
- renumbered Q5 to Q1
Connections:
- U3 pad 3: Net-(U3-XB) -> unconnected-(U3-XB-Pad3)
- Y2 pad 1: Net-(U3-XB) -> unconnected-(Y2-NC-Pad1)
- Y2 pad 3: Net-(U3-XA) -> Net-(Y2-OUT)
- Y2 pad 4: GND -> +3.3V
Routing:
- net +3.3V: track 55.3 -> 62.3 mm
- net GND: track 33.2 -> 38.2 mm, vias 146 -> 140
- net Net-(U3-XB): track 2.65 -> 0.00 mm
- net Net-(U3-XA): track 4.73 -> 2.37 mm
- net Net-(Y2-OUT): track 0.00 -> 1.89 mm
- net SDA: track 22.4 -> 21.8 mm
Other:
- board text added: "26MHz"
- board text added: "ptSolarHF Tracker v2.0.0 Custom Digital Services, LLC www.custom-ds.com"
- board text removed: "ptSolarHF Tracker v1.0.1 Custom Digital Services, LLC www.custom-ds.com"
