File: ptSolarHF/ptSolarHF.kicad_sch (KiCad schematic)
At the start: 55 parts, among them J1 6 Pin Male Header, J2 Programming, Q5 DMP2004K-7, U1 LP3985IM5-3.3/NOPB, U2 ATMega 328p-AU, U3 Si5351A-B-GT, U4 ATGM336H-5N31, U5 APX803S (SOT23SA), Y1 8MHz, Y2 Crystal_GND24

Commit message: Testing wspr_enc.c
Parts:
- U3: Digikey (none) -> 336-2399-5-ND
- Y2: value Crystal_GND24 -> 27MHz Xtal - 7M-27.000MEEQ-T; Digikey (none) -> 887-1328-1-ND
Changed lines of the file:
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@@
 			)
 		)
-		(property "Value" "Crystal_GND24"
+		(property "Value" "27MHz Xtal - 7M-27.000MEEQ-T"
 			(at 233.934 80.264 90)
 			(effects
@@
 		(property "Description" "Four pin crystal, GND on pins 2 and 4"
 			(at 234.95 86.36 0)
+			(effects
+				(font
+					(size 1.27 1.27)
+				)
+				(hide yes)
+			)
+		)
+		(property "Digikey" "887-1328-1-ND"
+			(at 234.95 86.36 90)
 			(effects
 				(font
@@
 			(at 264.16 91.44 0)
 			(effects
+				(font
+					(size 1.27 1.27)
+				)
+				(hide yes)
+			)
+		)
+		(property "Digikey" "  336-2399-5-ND"
+			(at 264.16 91.44 0)
+			(effects

Commit message: Tweaks to proof of concept. Updates to Schematics.
Parts:
- added C15: 100nF, Capacitor_SMD:C_0805_2012Metric, symbol Device:C
- added R10: 150k, Resistor_SMD:R_0805_2012Metric, symbol Device:R_US
- C16, C19: value 54pF -> 150pF; Digikey (none) -> 490-3315-1-ND
- C17, C18: Digikey (none) -> 490-1616-1-ND
- L1: value 381nH -> 270nF; Digikey (none) -> 490-5671-1-ND
- L2: value 612nH -> 270nH; Digikey (none) -> 490-5671-1-ND
- L3: value 381nH -> 270nH; Digikey (none) -> 490-5671-1-ND
- renumbered C14 to C13, C13 to C14, R23 to R11
Connections:
- net GND: now also R10.1
- net at ANT2.1 (In), ANT2a1.1 (Pin_1), C19.2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: now also R10.2
- net at C16.2, L1.1: now also C15.2; no longer U3.10 (CLK0)
- new net: C15.1, U3.10 (CLK0)
Other:
- moved on the sheet: ANT2, ANT2a1, ANT2b1, C16, C17, C18, C19, L1, L2, L3

Commit message: Implementing fine altitude modulation.
Parts:
- added C22: 1000pF, Capacitor_SMD:C_0805_2012Metric, symbol Device:C
- added C23: 100pF, Capacitor_SMD:C_0805_2012Metric, symbol Device:C
Changed lines of the file:
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@@
 	(wire
 		(pts
-			(xy 266.7 73.66) (xy 266.7 74.93)
+			(xy 266.7 60.96) (xy 266.7 74.93)
 		)
 		(stroke
@@
 	(symbol
 		(lib_id "power:+3.3V")
-		(at 266.7 73.66 0)
+		(at 266.7 60.96 0)
 		(unit 1)
 		(exclude_from_sim no)
@@
 		(fields_autoplaced yes)
 		(property "Reference" "#PWR05"
-			(at 266.7 77.47 0)
+			(at 266.7 64.77 0)
 			(effects
 				(font
@@
 		)
 		(property "Value" "+3.3V"
-			(at 266.7 68.58 0)
+			(at 266.7 55.88 0)
 			(effects
 				(font
@@
 		)
 		(property "Footprint" ""
-			(at 266.7 73.66 0)
+			(at 266.7 60.96 0)
 			(effects
 				(font
@@
 		)
 		(property "Datasheet" ""
-			(at 266.7 73.66 0)
+			(at 266.7 60.96 0)
 			(effects
 				(font
@@
 		)
 		(property "Description" "Power symbol creates a global label with name \"+3.3V\""
-			(at 266.7 73.66 0)
+			(at 266.7 60.96 0)
 			(effects
 				(font
@@
 	)
 	(symbol
+		(lib_id "Device:C")
+		(at 287.02 69.85 0)
+		(unit 1)
+		(exclude_from_sim no)
+		(in_bom yes)
+		(on_board yes)
+		(dnp no)
+		(property "Reference" "C23"
+			(at 288.036 69.215 0)
+			(effects
+				(font
+					(size 1.778 1.5113)
+				)
+				(justify left bottom)
+			)
+		)
+		(property "Value" "100pF"
+			(at 288.036 74.041 0)
+			(effects
+				(font
+					(size 1.778 1.5113)
+				)
+				(justify left bottom)
+			)
+		)
+		(property "Footprint" "Capacitor_SMD:C_0805_2012Metric"
+			(at 287.9852 73.66 0)
+			(effects
+				(font
+					(size 1.27 1.27)
+				)
+				(hide yes)
+			)
+		)
+		(property "Datasheet" "~"
+			(at 287.02 69.85 0)
+			(effects
+				(font
+					(size 1.27 1.27)
+				)
+				(hide yes)
+			)
+		)
+		(property "Description" "Unpolarized capacitor"
+			(at 287.02 69.85 0)
+			(effects
+				(font
+					(size 1.27 1.27)
+				)
+				(hide yes)
+			)
+		)
+		(property "Digikey" "399-17420-2-ND"
+			(at 287.02 69.85 0)
+			(effects
+				(font
+					(size 1.27 1.27)
+				)
+				(justify left bottom)
+				(hide yes)
+			)
+		)
+		(property "LCSC" ""
+			(at 287.02 69.85 0)
+			(effects
+				(font
+					(size 1.27 1.27)
+				)
+				(hide yes)
+			)
+		)
+		(pin "1"
+		)
+		(pin "2"
+		)
+		(instances
+			(project "ptSolarHF"
+				(path "/166d0a8f-2333-4a81-bfd6-a1b5ff84420a"
+					(reference "C23")
+					(unit 1)
+				)
+			)
+		)
+	)
+	(symbol
 		(lib_id "power:GND")
 		(at 355.6 99.06 0)
@@
 					(unit 1)
 				)
+			)
+		)
+	)
+	(symbol
+		(lib_id "Device:C")
+		(at 278.13 69.85 0)
+		(unit 1)
+		(exclude_from_sim no)
+		(in_bom yes)
+		(on_board yes)
+		(dnp no)
+		(property "Reference" "C22"
+			(at 279.146 69.215 0)
+			(effects
+				(font
+					(size 1.778 1.5113)
+				)
+				(justify left bottom)
+			)
+		)
+		(property "Value" "1000pF"
+			(at 279.146 74.041 0)
+			(effects
+				(font
+					(size 1.778 1.5113)
+				)
+				(justify left bottom)
+			)
+		)
+		(property "Footprint" "Capacitor_SMD:C_0805_2012Metric"
+			(at 279.0952 73.66 0)
+			(effects
+				(font
+					(size 1.27 1.27)
+				)
+				(hide yes)
+			)
+		)
+		(property "Datasheet" "~"
+			(at 278.13 69.85 0)
+			(effects
+				(font
+					(size 1.27 1.27)
+				)
+				(hide yes)
+			)
+		)
+		(property "Description" "Unpolarized capacitor"
+			(at 278.13 69.85 0)
+			(effects
+				(font
+					(size 1.27 1.27)
+				)
+				(hide yes)
+			)
+		)
+		(property "Digikey" "399-15433-2-ND"
+			(at 278.13 69.85 0)
+			(effects
+				(font
+					(size 1.27 1.27)
+				)
+				(justify left bottom)
+				(hide yes)
+			)
+		)
+		(property "LCSC" ""
+			(at 278.13 69.85 0)
+			(effects
+				(font
+					(size 1.27 1.27)
+				)
+				(hide yes)
+			)
+		)
+		(pin "1"
+		)
+		(pin "2"
+		)
+		(instances
+			(project "ptSolarHF"
+				(path "/166d0a8f-2333-4a81-bfd6-a1b5ff84420a"
+					(reference "C22")
+					(unit 1)
+				)

Commit message: Finalizing PCB v1.0.1
Parts:
- removed ANT2a1, ANT2b1: VHF Test Point, Custom DS:Small Test Point Pin, symbol Connector_Generic:Conn_01x01
- removed C22: 1000pF, Capacitor_SMD:C_0805_2012Metric, symbol Device:C
- removed C23: 100pF, Capacitor_SMD:C_0805_2012Metric, symbol Device:C
- C1: value 6V 1F -> 6V 0.5F; Digikey 4688-CSP-6R0L105R-TW-ND -> 4688-CSP-6R0L504R-TW-ND
- C15: LCSC (none) -> C49678
- C16, C19: value 150pF -> 180pF; Digikey 490-3315-1-ND -> 490-11541-1-ND; LCSC (none) -> C113826
- C17, C18: value 220pF -> 270pF; Digikey 490-1616-1-ND -> 490-9738-1-ND; LCSC (none) -> C527183
- L1: value 270nF -> 330nH; Digikey 490-5671-1-ND -> 490-5672-1-ND; LCSC (none) -> C184530
- L2: value 270nH -> 390nH; Digikey 490-5671-1-ND -> 490-5673-1-ND; LCSC (none) -> C108076
- L3: value 270nH -> 330nH; Digikey 490-5671-1-ND -> 490-5672-1-ND; LCSC (none) -> C184530
- R10: value 150k -> 10k; Digikey 311-150KCRCT-ND -> 13-RT0805FRD0710KLCT-ND; LCSC C114558 -> C100047
- U3: Digikey 336-2399-5-ND -> 336-2399-5-ND; LCSC (none) -> C504891
- Y2: LCSC (none) -> C2450429
